Commit message: first success of full urdf

File: exo_fri/urdf/exo_fri.urdf (robot description, URDF)
Before this commit: robot thormang3, 13 links, 12 joints
Links:
- link l_leg_an_p_link: mass 0.0325752774497041 -> 0.032575; geometry collision mesh filename=package://exo_fri/meshes/l_leg_an_p_link.STL; visual mesh filename=package://exo_fri/meshes/l_leg_an_p_link.STL
- link l_leg_an_r_link: mass 2.0447635642258 -> 0.204476356422574; geometry collision mesh filename=package://exo_fri/meshes/l_leg_an_r_link.STL; visual mesh filename=package://exo_fri/meshes/l_leg_an_r_link.STL
- link l_leg_hip_p_link: mass 0.286678540994592 -> 0.28668; geometry collision mesh filename=package://exo_fri/meshes/l_leg_hip_p_link.STL; visual mesh filename=package://exo_fri/meshes/l_leg_hip_p_link.STL
- link l_leg_hip_r_link: mass 0.577322605082582 -> 0.577322605082581; geometry collision mesh filename=package://exo_fri/meshes/l_leg_hip_r_link.STL; visual mesh filename=package://exo_fri/meshes/l_leg_hip_r_link.STL
- link l_leg_hip_y_link: mass 0.0865282088524624 -> 0.086528; geometry collision mesh filename=package://exo_fri/meshes/l_leg_hip_y_link.STL; visual mesh filename=package://exo_fri/meshes/l_leg_hip_y_link.STL
- link l_leg_kn_p_link: mass 0.501847265279983 -> 0.50185; geometry collision mesh filename=package://exo_fri/meshes/l_leg_kn_p_link.STL; visual mesh filename=package://exo_fri/meshes/l_leg_kn_p_link.STL
- link pelvis_link: geometry collision mesh filename=package://exo_fri/meshes/pelvis_link.STL; visual mesh filename=package://exo_fri/meshes/pelvis_link.STL
- link r_leg_an_p_link: geometry collision mesh filename=package://exo_fri/meshes/r_leg_an_p_link.STL; visual mesh filename=package://exo_fri/meshes/r_leg_an_p_link.STL
- link r_leg_an_r_link: mass 1.99852541528706 -> 0.199852541528696; geometry collision mesh filename=package://exo_fri/meshes/r_leg_an_r_link.STL; visual mesh filename=package://exo_fri/meshes/r_leg_an_r_link.STL
- link r_leg_hip_p_link: geometry collision mesh filename=package://exo_fri/meshes/r_leg_hip_p_link.STL; visual mesh filename=package://exo_fri/meshes/r_leg_hip_p_link.STL
- link r_leg_hip_r_link: geometry collision mesh filename=package://exo_fri/meshes/r_leg_hip_r_link.STL; visual mesh filename=package://exo_fri/meshes/r_leg_hip_r_link.STL
- link r_leg_hip_y_link: geometry collision mesh filename=package://exo_fri/meshes/r_leg_hip_y_link.STL; visual mesh filename=package://exo_fri/meshes/r_leg_hip_y_link.STL
- link r_leg_kn_p_link: mass 0.501848142816981 -> 0.501848142816943; geometry collision mesh filename=package://exo_fri/meshes/r_leg_kn_p_link.STL; visual mesh filename=package://exo_fri/meshes/r_leg_kn_p_link.STL
Joints:
- joint r_leg_hip_r: origin xyz=0 0 0 rpy=0 0 0 -> xyz=0 -0.25 0 rpy=0 0 0
- joint r_leg_hip_y: origin xyz=0.023 -0.125 -0.0813 rpy=0 0 0 -> xyz=0.023 0.125 -0.0813 rpy=0 0 0
