Commit message: first walk in simulation

File: all_exo_new_urdf_7_4/urdf/all_exo_new_urdf_7_4.xacro (robot description, xacro)
@@ -415,4 +415,20 @@
   </joint>
 <xacro:insert_transmission name="l_leg_an_r" />
+  <!-- left ft joint -->
+  <joint name="l_leg_ft" type="revolute">
+    <origin xyz="-0.057 0.0 -0.087" rpy="0 0 0"/>
+    <parent link="l_leg_an_r_link"/>
+    <child link="l_leg_foot_link"/>
+    <limit velocity="6.5" effort="1000" lower="0" upper="0" />
+  </joint>
+  <!-- left foot link -->
+  <link name="l_leg_foot_link">
+    <inertial>
+    <origin xyz="0.000 0.009 -0.013" rpy="0 0 0"/>
+    <mass value="0.1689"/>
+    <inertia ixx="1.0" ixy="0.0" ixz="0.0" iyy="1.0" iyz="0.0" izz="1.0" />
+    <!-- <inertia ixx="0.00219" ixy="0.0" ixz="0.0" iyy="0.00433" iyz="0.00011" izz="0.00609" /> -->
+    </inertial>
+  </link>
   <link
     name="r_leg_hip_y_link">
@@ -787,4 +803,20 @@
   </joint>
 <xacro:insert_transmission name="r_leg_an_r" />
+  <!-- left ft joint -->
+  <joint name="r_leg_ft" type="revolute">
+    <origin xyz="-0.057 0.0 -0.087" rpy="0 0 0"/>
+    <parent link="r_leg_an_r_link"/>
+    <child link="r_leg_foot_link"/>
+    <limit velocity="6.5" effort="1000" lower="0" upper="0" />
+  </joint>
+  <!-- left foot link -->
+  <link name="r_leg_foot_link">
+    <inertial>
+    <origin xyz="0.000 0.009 -0.013" rpy="0 0 0"/>
+    <mass value="0.1689"/>
+    <inertia ixx="1.0" ixy="0.0" ixz="0.0" iyy="1.0" iyz="0.0" izz="1.0" />
+    <!-- <inertia ixx="0.00219" ixy="0.0" ixz="0.0" iyy="0.00433" iyz="0.00011" izz="0.00609" /> -->
+    </inertial>
+  </link>
     <!-- ros_control plugin -->
   <gazebo>
